File: in_out.kicad_sch (KiCad schematic)
At the start: 22 parts, among them J2 Micro_SD_Card_Det1, J3 Conn_01x10, SW1 SW_Push, SW2 SW_Push, U5 DM-OLED096-636

Commit message: set initial component footprints
Parts:
- J2: renamed from J3; footprint (none) -> Connector_PinSocket_2.54mm:PinSocket_1x10_P2.54mm_Horizontal
- R13: renamed from R8; footprint (none) -> Resistor_SMD:R_0603_1608Metric
- R14: renamed from R9; footprint (none) -> Resistor_SMD:R_0603_1608Metric
- R15: renamed from R10; footprint (none) -> Resistor_SMD:R_0603_1608Metric
- R16: renamed from R11; footprint (none) -> Resistor_SMD:R_0603_1608Metric
- R17: renamed from R12; footprint (none) -> Resistor_SMD:R_0603_1608Metric
- R18: renamed from R13; footprint (none) -> Resistor_SMD:R_0603_1608Metric
- R19: renamed from R14; footprint (none) -> Resistor_SMD:R_0603_1608Metric
- R20: renamed from R15; footprint (none) -> Resistor_SMD:R_0603_1608Metric
- R21: renamed from R2; footprint (none) -> Resistor_SMD:R_0603_1608Metric
- R22: renamed from R3; footprint (none) -> Resistor_SMD:R_0603_1608Metric
- R23: renamed from R5; footprint (none) -> Resistor_SMD:R_0603_1608Metric
- R24: renamed from R6; footprint (none) -> Resistor_SMD:R_0603_1608Metric
- R25: renamed from R7; footprint (none) -> Resistor_SMD:R_0603_1608Metric
- renumbered D3 to D5, D4 to D6, D2 to D7, J2 to J3, U5 to U6

Commit message: Add footprints
Parts:
- BZ1: footprint (none) -> Buzzer_Beeper:Buzzer_CUI_CPT-9019S-SMT
- SW1, SW2: footprint (none) -> Button_Switch_SMD:SW_SPST_SKQG_WithoutStem
Changed lines of the file:
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@@
 			)
 		)
-		(property "Footprint" ""
+		(property "Footprint" "Button_Switch_SMD:SW_SPST_SKQG_WithoutStem"
 			(at 158.75 78.74 0)
 			(effects
@@
 			)
 		)
-		(property "Footprint" ""
+		(property "Footprint" "Buzzer_Beeper:Buzzer_CUI_CPT-9019S-SMT"
 			(at 205.105 133.35 90)
 			(effects
@@
 			)
 		)
-		(property "Footprint" ""
+		(property "Footprint" "Button_Switch_SMD:SW_SPST_SKQG_WithoutStem"
 			(at 158.75 59.69 0)
 			(effects

Commit message: Initial pcb component placement
Parts:
- J3: footprint (none) -> microsd:TF-SMD_A-MICROTF-1.85A
Changed lines of the file:
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@@
 			)
 		)
-		(property "Footprint" ""
+		(property "Footprint" "microsd:TF-SMD_A-MICROTF-1.85A"
 			(at 162.56 52.07 0)
 			(effects
