File: in_out.kicad_sch (KiCad schematic)
At the start: 25 parts, among them J2 Conn_01x08, J3 Micro_SD_Card_Det1, Q3 NMOS, SW1 SW_Push, SW2 SW_Push, U6 DM-OLED096-636

Commit message: LUIGI
Parts:
- C25: value C -> 10u
- R13: value R_Small -> 100
- R14, R15, R16, R17, R18: value R_Small -> 100R
- R21: value R -> 10k
- R22: value R -> 20k
- R23, R24, R25: value R -> 100
Changed lines of the file:
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@@
 			)
 		)
-		(property "Value" "R_Small"
+		(property "Value" "100R"
 			(at 160.02 109.22 90)
 			(effects
@@
 			)
 		)
-		(property "Value" "R"
+		(property "Value" "10k"
 			(at 170.18 62.484 90)
 			(effects
@@
 		(dnp no)
 		(property "Reference" "R24"
-			(at 194.056 114.046 90)
-			(effects
-				(font
-					(size 1.27 1.27)
-				)
-			)
-		)
-		(property "Value" "R"
-			(at 197.104 114.046 90)
+			(at 195.58 109.728 90)
+			(effects
+				(font
+					(size 1.27 1.27)
+				)
+			)
+		)
+		(property "Value" "100"
+			(at 195.58 114.046 90)
 			(effects
 				(font
@@
 			)
 		)
-		(property "Value" "R_Small"
+		(property "Value" "100R"
 			(at 160.02 124.46 90)
 			(effects
@@
 			)
 		)
-		(property "Value" "R_Small"
+		(property "Value" "100R"
 			(at 160.02 116.84 90)
 			(effects
@@
 			)
 		)
-		(property "Value" "R"
+		(property "Value" "100"
 			(at 195.58 104.394 90)
 			(effects
@@
 			)
 		)
-		(property "Value" "R"
+		(property "Value" "20k"
 			(at 170.18 81.534 90)
 			(effects
@@
 			)
 		)
-		(property "Value" "R_Small"
+		(property "Value" "100R"
 			(at 160.02 113.03 90)
 			(effects
@@
 			)
 		)
-		(property "Value" "R"
+		(property "Value" "100"
 			(at 195.58 121.666 90)
 			(effects
@@
 			)
 		)
-		(property "Value" "R_Small"
+		(property "Value" "100R"
 			(at 160.02 120.65 90)
 			(effects
@@
 			)
 		)
-		(property "Value" "C"
+		(property "Value" "10u"
 			(at 69.85 71.1199 0)
 			(effects
@@
 			)
 		)
-		(property "Value" "R_Small"
+		(property "Value" "100"
 			(at 160.02 105.41 90)
 			(effects
