File: mcu.kicad_sch (KiCad schematic)
At the start: 3 parts, among them U1 ESP32-S3-WROOM-1

Commit message: set initial component footprints
Parts:
- C5: renamed from C1; footprint (none) -> Capacitor_SMD:C_0603_1608Metric
- C6: renamed from C2; footprint (none) -> Capacitor_SMD:C_0603_1608Metric
- renumbered U1 to U4
Changed lines of the file:
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@@
 		(on_board yes)
 		(dnp no)
-		(property "Reference" "#PWR03"
+		(property "Reference" "#PWR011"
 			(at 26.67 33.02 0)
 			(effects
@@
 			(project "pipu-zero"
 				(path "/3130e1f2-bde1-4b12-bd54-0e1e50bd36da/2c03e026-3c91-4c99-bc42-f7cc422549b7"
-					(reference "#PWR03")
+					(reference "#PWR011")
 					(unit 1)
 				)
@@
 		(dnp no)
 		(fields_autoplaced yes)
-		(property "Reference" "U1"
+		(property "Reference" "U4"
 			(at 110.0933 25.4 0)
 			(effects
@@
 			(project "pipu-zero"
 				(path "/3130e1f2-bde1-4b12-bd54-0e1e50bd36da/2c03e026-3c91-4c99-bc42-f7cc422549b7"
-					(reference "U1")
+					(reference "U4")
 					(unit 1)
 				)
@@
 		(on_board yes)
 		(dnp no)
-		(property "Reference" "C1"
+		(property "Reference" "C5"
 			(at 29.21 34.29 0)
 			(effects
@@
 			)
 		)
-		(property "Footprint" ""
+		(property "Footprint" "Capacitor_SMD:C_0603_1608Metric"
 			(at 27.6352 39.37 0)
 			(effects
@@
 			(project ""
 				(path "/3130e1f2-bde1-4b12-bd54-0e1e50bd36da/2c03e026-3c91-4c99-bc42-f7cc422549b7"
-					(reference "C1")
+					(reference "C5")
 					(unit 1)
 				)
@@
 		(on_board yes)
 		(dnp no)
-		(property "Reference" "C2"
+		(property "Reference" "C6"
 			(at 39.37 34.29 0)
 			(effects
@@
 			)
 		)
-		(property "Footprint" ""
+		(property "Footprint" "Capacitor_SMD:C_0603_1608Metric"
 			(at 37.7952 39.37 0)
 			(effects
@@
 			(project "pipu-zero"
 				(path "/3130e1f2-bde1-4b12-bd54-0e1e50bd36da/2c03e026-3c91-4c99-bc42-f7cc422549b7"
-					(reference "C2")
+					(reference "C6")
 					(unit 1)
 				)
@@
 		(on_board yes)
 		(dnp no)
-		(property "Reference" "#PWR02"
+		(property "Reference" "#PWR014"
 			(at 107.95 29.21 0)
 			(effects
@@
 			(project ""
 				(path "/3130e1f2-bde1-4b12-bd54-0e1e50bd36da/2c03e026-3c91-4c99-bc42-f7cc422549b7"
-					(reference "#PWR02")
+					(reference "#PWR014")
 					(unit 1)
 				)
@@
 		(on_board yes)
 		(dnp no)
-		(property "Reference" "#PWR05"
+		(property "Reference" "#PWR013"
 			(at 83.82 35.56 0)
 			(effects
@@
 			(project ""
 				(path "/3130e1f2-bde1-4b12-bd54-0e1e50bd36da/2c03e026-3c91-4c99-bc42-f7cc422549b7"
-					(reference "#PWR05")
+					(reference "#PWR013")
 					(unit 1)
 				)
@@
 		(on_board yes)
 		(dnp no)
-		(property "Reference" "#PWR01"
+		(property "Reference" "#PWR015"
 			(at 107.95 91.44 0)
 			(effects
@@
 			(project ""
 				(path "/3130e1f2-bde1-4b12-bd54-0e1e50bd36da/2c03e026-3c91-4c99-bc42-f7cc422549b7"
-					(reference "#PWR01")
+					(reference "#PWR015")
 					(unit 1)
 				)
@@
 		(on_board yes)
 		(dnp no)
-		(property "Reference" "#PWR04"
+		(property "Reference" "#PWR012"
 			(at 26.67 48.26 0)
 			(effects
@@
 			(project ""
 				(path "/3130e1f2-bde1-4b12-bd54-0e1e50bd36da/2c03e026-3c91-4c99-bc42-f7cc422549b7"
-					(reference "#PWR04")
-					(unit 1)
-				)
+					(reference "#PWR012")
+					(unit 1)
+				)

Commit message: modify ios
Parts:
- added Q4: NMOS, Package_TO_SOT_SMD:SOT-23, symbol Transistor_FET:Q_NMOS_GSD
Connections:
- net IO0 is gone; now on net BTN1: U4.27 (IO0)
- net IO14 is gone; now on net IR_RX: U4.22 (IO14)
- net IO3 is gone; now on net BTN2: U4.15 (IO3)
- net IO38 is gone; now on net BUZZER: U4.31 (IO38)
- net BTN1: no longer U4.26 (IO45)
- net BTN2: no longer U4.35 (IO42)
- net BUZZER: no longer U4.32 (IO39)
- net GND: now also Q4.2 (S)
- net IR_RX: no longer U4.33 (IO40)
- net IR_TX: now also Q4.3 (D); no longer U4.34 (IO41)
- net IO46: no longer names the net of U4.16 (IO46)
- net IO9: no longer names the net of U4.17 (IO9)
- net RGB_R: no longer names the net of U4.23 (IO21)
- net RGB_R: now also Q4.1 (G)
- new net IO39: U4.32 (IO39)
- new net IO40: U4.33 (IO40)
- new net IO41: U4.34 (IO41)
- new net IO42: U4.35 (IO42)
