File: pipu-zero.kicad_pcb (KiCad board)
At the start: 2 copper layers, 40 x 70 mm, 75 parts, among them IC1 BQ25176JDSGR, J1 USB_C_Receptacle_USB2.0_14P, J2 Conn_01x10, J3 Micro_SD_Card_Det1, Q1 NMOS, Q2 NMOS, SW1 SW_Push, SW2 SW_Push, U1 BQ297xy, U2 MCP1640Bx-xCHY, U3 MCP1727-0802xSN, U4 ESP32-S3-WROOM-1, U5 CC1101, U6 DM-OLED096-636, U7 TSOP348xx, Y2 Crystal_GND23

Commit message: update pcb and schematic
Parts:
- removed R19, R20: R_Small, Resistor_SMD:R_0603_1608Metric
- added Q3: NMOS, Package_TO_SOT_SMD:SOT-23, F.Cu at (45.0, 105.7)
- added Q4: NMOS, Package_TO_SOT_SMD:SOT-23, F.Cu at (31.1, 60.2)
- BZ1, C2, Q1: moved to B.Cu
- J2: value Conn_01x10 -> Conn_01x08; footprint Connector_PinSocket_2.54mm:PinSocket_1x10_P2.54mm_Horizontal -> Connector_PinSocket_2.54mm:PinSocket_1x08_P2.54mm_Horizontal
- moved SW2 195.5 mm to (229.5, 62.5)
- moved BZ1 185.3 mm to (198.5, 41.0)
- moved SW1 184.8 mm to (219.0, 58.0)
- moved D7 176.8 mm to (219.0, 67.0)
- moved U5 133.9 mm to (219.2, 42.5)
- moved D4 133.2 mm to (204.0, 25.0), turned to 180 degrees
- moved J3 127.6 mm to (169.0, 66.5)
- moved U7 121.6 mm to (198.1, 24.7), turned to 180 degrees
- moved U4 121.0 mm to (165.1, 45.9), turned to 90 degrees
- moved U3 119.6 mm to (91.9, 77.2), turned to 0 degrees
- moved D2 108.7 mm to (94.5, 82.0)
- moved D3 108.7 mm to (94.5, 85.0)
- moved R4 108.7 mm to (81.5, 81.8)
- moved R5 108.7 mm to (81.5, 84.3)
- moved R6 108.7 mm to (81.5, 86.8)
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Connections:
- BZ1 pad 1: /I-O/BUZZER -> +3V3
- BZ1 pad 2: GND -> Net-(BZ1--)
- D4 pad 1: GND -> Net-(D4-K)
- D4 pad 2: Net-(D4-A) -> +3V3
- D5 pad 1: /I-O/IO46 -> /I-O/IO39_EXT
- D5 pad 3: /I-O/IO38 -> /I-O/IO40_EXT
- D5 pad 4: /I-O/IO14 -> /I-O/IO41_EXT
- D5 pad 6: /I-O/IO9 -> /I-O/IO42_EXT
- D6 pad 1: /I-O/IO3 -> unconnected-(D6-TVS1-Pad1)
- D6 pad 3: /I-O/IO0 -> unconnected-(D6-TVS2-Pad3)
- D7 pad 2: GND -> /I-O/RGB_B
- D7 pad 4: GND -> /I-O/RGB_G
- D7 pad 6: GND -> /I-O/RGB_R
- J2 pad 2: /I-O/IO46_EXT -> /I-O/IO42_EXT
- J2 pad 3: /I-O/IO38_EXT -> /I-O/IO41_EXT
- J2 pad 4: /I-O/IO14_EXT -> /I-O/IO40_EXT
- J2 pad 5: /I-O/IO9_EXT -> /I-O/IO39_EXT
- J2 pad 6: /I-O/IO3_EXT -> /I-O/TXD0_EXT
- J2 pad 7: /I-O/IO0_EXT -> /I-O/RXD0_EXT
- J2 pad 8: /I-O/TXD0_EXT -> GND
- R11 pad 1: /Infrared/IR_TX -> /I-O/RGB_B
- R11 pad 2: Net-(D4-A) -> Net-(D4-K)
- R15 pad 1: /I-O/IO0 -> /I-O/IO39
- R15 pad 2: /I-O/IO0_EXT -> /I-O/IO39_EXT
- R16 pad 1: /I-O/IO3 -> /I-O/IO40
- R16 pad 2: /I-O/IO3_EXT -> /I-O/IO40_EXT
- R17 pad 1: /I-O/IO9 -> /I-O/IO41
- R17 pad 2: /I-O/IO9_EXT -> /I-O/IO41_EXT
- R18 pad 1: /I-O/IO14 -> /I-O/IO42
- R18 pad 2: /I-O/IO14_EXT -> /I-O/IO42_EXT
- R23 pad 1: /I-O/RGB_B -> +3V3
- R24 pad 1: /I-O/RGB_G -> +3V3
- R25 pad 1: /I-O/RGB_R -> +3V3
- U4 pad 15: /I-O/IO3 -> /I-O/BTN2
- U4 pad 16: /I-O/IO46 -> unconnected-(U4-IO46-Pad16)
- U4 pad 17: /I-O/IO9 -> unconnected-(U4-IO9-Pad17)
- U4 pad 22: /I-O/IO14 -> /Infrared/IR_RX
- U4 pad 23: /I-O/RGB_B -> Net-(Q4-G)
- U4 pad 26: /I-O/BTN1 -> unconnected-(U4-IO45-Pad26)
- U4 pad 27: /I-O/IO0 -> /I-O/BTN1
- U4 pad 31: /I-O/IO38 -> /I-O/BUZZER
- U4 pad 32: /I-O/BUZZER -> /I-O/IO39
- U4 pad 33: /Infrared/IR_RX -> /I-O/IO40
- U4 pad 34: /Infrared/IR_TX -> /I-O/IO41
- U4 pad 35: /I-O/BTN2 -> /I-O/IO42
Other:
- board size 40 x 70 mm -> 80 x 50.5 mm
- copper layers 2 -> 4

Commit message: update pcb and schematic
Parts:
- added C21: C, Capacitor_SMD:C_0805_2012Metric, F.Cu at (42.4, 164.6)
- added C22: C, Capacitor_SMD:C_0805_2012Metric, F.Cu at (42.4, 167.6)
- added C23: C, Capacitor_SMD:C_0805_2012Metric, F.Cu at (48.9, 164.6)
- added C24: C, Capacitor_SMD:C_0805_2012Metric, F.Cu at (48.9, 167.6)
- added C25: C, Capacitor_SMD:C_0805_2012Metric, B.Cu at (169.1, 61.5)
- added U8: ~, Encoder:encoder, F.Cu at (231.5, 29.2)
- C1, D1, D5, D6, L1, R10, R23, R24, R25, R5, R6: moved to B.Cu
- C10, C13, C8: footprint Capacitor_SMD:C_0603_1608Metric -> Capacitor_SMD:C_0402_1005Metric; moved to B.Cu
- C12, C14, C15, C7, C9: footprint Capacitor_SMD:C_0603_1608Metric -> Capacitor_SMD:C_0402_1005Metric
- moved C20 157.8 mm to (218.3, 27.8)
- moved C13 156.8 mm to (220.2, 41.5), turned to -90 degrees
- moved R21 156.2 mm to (227.5, 58.0), turned to 90 degrees
- moved R22 156.0 mm to (227.5, 65.0), turned to 90 degrees
- moved C9 154.4 mm to (220.7, 38.5)
- moved C15 154.2 mm to (225.5, 38.5)
- moved C12 153.8 mm to (216.7, 38.5), turned to 180 degrees
- moved C19 152.8 mm to (215.0, 29.5), turned to 180 degrees
- moved C10 151.8 mm to (216.8, 38.5), turned to 180 degrees
- moved C17 151.7 mm to (219.5, 35.7), turned to 90 degrees
- moved C14 151.3 mm to (225.5, 45.0)
- moved C8 150.1 mm to (218.7, 43.0), turned to 180 degrees
- moved C18 150.0 mm to (215.0, 33.0), turned to 180 degrees
- moved L5 148.8 mm to (217.6, 30.3), turned to 90 degrees
- moved R24 148.5 mm to (218.0, 49.5)
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Connections:
- U4 pad 16: unconnected-(U4-IO46-Pad16) -> /I-O/ENCODER_C
- U4 pad 17: unconnected-(U4-IO9-Pad17) -> /I-O/ENCODER_A
- U4 pad 26: unconnected-(U4-IO45-Pad26) -> /I-O/ENCODER_B
