File: pipu-zero.kicad_sch (KiCad schematic)
At the start: 4 parts, among them J1 USB_C_Receptacle_USB2.0_14P

Commit message: add cc1101 passives
Parts:
- R1, R2: value R_Small -> 5.1k
Changed lines of the file:
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@@
 			)
 		)
-		(property "Value" "R_Small"
+		(property "Value" "5.1k"
 			(at 50.8 102.87 90)
 			(effects
@@
 			)
 		)
-		(property "Value" "R_Small"
+		(property "Value" "5.1k"
 			(at 50.8 105.41 90)
 			(effects
