File: radio.kicad_sch (KiCad schematic)
At the start: 22 parts, among them U5 CC1101, Y2 X322526MMB4SI

Commit message: LUIGI
Parts:
- AE1: footprint Connector_PinHeader_2.54mm:PinHeader_1x01_P2.54mm_Vertical -> (none)
Changed lines of the file:
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@@
 			)
 		)
-		(property "Footprint" "Connector_PinHeader_2.54mm:PinHeader_1x01_P2.54mm_Vertical"
+		(property "Footprint" ""
 			(at 219.71 129.54 0)
 			(effects
